File: pcb-right/pcb-right.kicad_sch (KiCad schematic)
At the start: 39 parts, among them J3 BAT, U2 xiao-ble

Commit message: Right Positioned
Parts:
- J3: footprint Connector_JST:JST_PH_S2B-PH-SM4-TB_1x02-1MP_P2.00mm_Horizontal -> Connector_PinHeader_2.54mm:PinHeader_1x02_P2.54mm_Vertical

Commit message: RC1
Parts:
- J3: now not fitted
Changed lines of the file:
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@@
 		(in_bom yes)
 		(on_board yes)
-		(dnp no)
+		(dnp yes)
 		(fields_autoplaced yes)
 		(property "Reference" "J3"
