File: pcb-right/pcb-right.kicad_pcb (KiCad board)
At the start: 2 copper layers, 124.8 x 104.5 mm, 43 parts, among them J2 BAT, U2 xiao-ble

Commit message: Right Positioned
Parts:
- J2: footprint Connector_JST:JST_PH_S2B-PH-SM4-TB_1x02-1MP_P2.00mm_Horizontal -> Connector_PinHeader_2.54mm:PinHeader_1x02_P2.54mm_Vertical
- moved SWR15 26.3 mm to (127.0, 84.5)
- moved SWR10 25.1 mm to (127.0, 67.5)
- moved SWR14 24.8 mm to (109.0, 70.0)
- moved SWR11 24.1 mm to (55.0, 72.5)
- moved SWR5 24.0 mm to (127.0, 50.5)
- moved SWR9 23.6 mm to (109.0, 53.0)
- moved SWR12 23.2 mm to (73.0, 70.0)
- moved SWR13 22.8 mm to (91.0, 65.8)
- moved SWR6 22.6 mm to (55.0, 55.5)
- moved SWR4 22.5 mm to (109.0, 36.0)
- moved SWR7 22.0 mm to (73.0, 53.0)
- moved SWR8 21.7 mm to (91.0, 48.8)
- moved SWR1 21.3 mm to (55.0, 38.5)
- moved SWR2 20.8 mm to (73.0, 36.0)
- moved SWR3 20.7 mm to (91.0, 31.8)
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Routing:
- net Net-(DR2-A): track 8.31 -> 184.8 mm
- net COL4_R: track 176.5 -> 0.00 mm
- net Net-(DR5-A): track 8.36 -> 170.8 mm
- net Net-(DR11-A): track 8.31 -> 156.2 mm
- net COL3_R: track 147.9 -> 0.00 mm
- net ROW3_R: track 190.7 -> 44.5 mm, vias 4 -> 0
- net GND_R: track 0.00 -> 78.1 mm, vias 29 -> 0
- net ROW2_R: track 165.8 -> 95.4 mm, vias 10 -> 0
- net ROW1_R: track 147.7 -> 115.0 mm, vias 10 -> 0
- net Net-(DR1-A): track 8.78 -> 35.0 mm
- net COL1_R: track 64.9 -> 89.8 mm
- net COL0_R: track 78.1 -> 57.7 mm
- net Net-(DR15-A): track 8.31 -> 19.6 mm
- net Net-(DR4-A): track 8.31 -> 0.00 mm
- net Net-(DR9-A): track 8.31 -> 0.00 mm
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Other:
- board size 124.8 x 104.5 mm -> 118.8 x 99.7 mm
- board text removed: "BAT +"
- board text removed: "BAT -"
- board text removed: "BATTERY"
- board text removed: "XIAO nRF52840"

Commit message: PCB v1
Parts:
- moved REF** 0.18 mm to (52.4, 91.2)
Routing:
- net Net-(DR2-A): track 184.8 -> 8.09 mm
- net Net-(DR5-A): track 170.8 -> 8.09 mm
- net COL4_R: track 0.00 -> 149.6 mm
- net Net-(DR11-A): track 156.2 -> 8.09 mm
- net COL3_R: track 0.00 -> 124.8 mm
- net GND_R: track 78.1 -> 202.4 mm
- net ROW3_R: track 44.5 -> 166.0 mm, vias 0 -> 2
- net VBAT_R: track 83.3 -> 116.1 mm
- net COL1_R: track 89.8 -> 59.0 mm
- net ROW2_R: track 95.4 -> 125.6 mm, vias 0 -> 5
- net Net-(DR1-A): track 35.0 -> 8.09 mm
- net ROW0_R: track 103.4 -> 89.4 mm, vias 0 -> 5
- net ROW1_R: track 115.0 -> 101.1 mm, vias 0 -> 5
- net Net-(DR15-A): track 19.6 -> 8.09 mm
- net COL0_R: track 57.7 -> 67.9 mm
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- removed copper zone on B.Cu, net GND_R
- removed copper zone on F.Cu, net GND_R
Other:
- outline, holes or cut-outs redrawn
- board text added: "${TITLE}"
- board text added: "+"
- board text added: "-"
- board text added: "Version ${REVISION} - ${CURRENT_DATE}"

Commit message: Long overdue commit!
Parts:
- moved REF** 0.23 mm to (52.5, 91.0)
Routing:
- added copper zone on B.Cu, net (none)
- added copper zone on F.Cu, net (none)
Changed lines of the file:
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@@
 		(pad_to_mask_clearance 0)
 		(allow_soldermask_bridges_in_footprints no)
-		(grid_origin 50.573343 101.496439)
+		(grid_origin 150 30)
 		(pcbplotparams
 			(layerselection 0x00010fc_ffffffff)
@@
 	)
 	(footprint "MountingHole:MountingHole_2.2mm_M2_DIN965_Pad"
-		(locked yes)
 		(layer "F.Cu")
-		(at 52.373343 91.196439)
+		(at 52.5 91)
 		(descr "Mounting Hole 2.2mm, M2, DIN965")
 		(tags "mounting hole 2.2mm m2 din965")
@@
 			)
 		)
-		(attr exclude_from_pos_files exclude_from_bom)
+		(attr board_only exclude_from_pos_files exclude_from_bom)
 		(fp_circle
 			(center 0 0)
@@
 	)
 	(footprint "MountingHole:MountingHole_2.2mm_M2_DIN965_Pad"
-		(locked yes)
 		(layer "F.Cu")
-		(at 123.75 32.49)
+		(at 123.75 32.5)
 		(descr "Mounting Hole 2.2mm, M2, DIN965")
 		(tags "mounting hole 2.2mm m2 din965")
@@
 			)
 		)
-		(attr exclude_from_pos_files exclude_from_bom)
+		(attr board_only exclude_from_pos_files exclude_from_bom)
 		(fp_circle
 			(center 0 0)
@@
 			(at 0 -2.33 -90)
 			(layer "F.SilkS")
+			(hide yes)
 			(effects
 				(font
@@
 	)
 	(footprint "MountingHole:MountingHole_2.2mm_M2_DIN965_Pad"
-		(locked yes)
 		(layer "F.Cu")
-		(at 147.5 106.74)
+		(at 147.5 106.7)
 		(descr "Mounting Hole 2.2mm, M2, DIN965")
 		(tags "mounting hole 2.2mm m2 din965")
@@
 			)
 		)
-		(attr exclude_from_pos_files exclude_from_bom)
+		(attr board_only exclude_from_pos_files exclude_from_bom)
 		(fp_circle
 			(center 0 0)
@@
 	)
 	(footprint "MountingHole:MountingHole_2.2mm_M2_DIN965_Pad"
-		(locked yes)
 		(layer "F.Cu")
 		(at 52.5 32.5)
@@
 			)
 		)
-		(attr exclude_from_pos_files exclude_from_bom)
+		(attr board_only exclude_from_pos_files exclude_from_bom)
 		(fp_circle
 			(center 0 0)
@@
 			(justify left bottom)
 		)
-		(render_cache "Version 1 - 2024-12-14" 0
+		(render_cache "Version 1 - 2024-12-16" 0
 			(polygon
 				(pts
@@
 			(polygon
 				(pts
-					(xy 106.707048 95.351281) (xy 106.835031 95.351281) (xy 106.835031 95.523228) (xy 106.707048 95.523228)
-					(xy 106.707048 95.726439) (xy 106.504326 95.726439) (xy 106.504326 95.523228) (xy 106.069574 95.523228)
-					(xy 106.069574 95.351281) (xy 106.2806 95.351281) (xy 106.504326 95.351281) (xy 106.504326 95.002991)
-					(xy 106.50164 95.002991) (xy 106.2806 95.351281) (xy 106.069574 95.351281) (xy 106.069574 95.345664)
-					(xy 106.476239 94.72602) (xy 106.707048 94.72602)
+					(xy 106.439602 95.095071) (xy 106.473308 95.088232) (xy 106.508479 95.085545) (xy 106.559449 95.089049)
+					(xy 106.610636 95.100751) (xy 106.636462 95.110458) (xy 106.680672 95.133683) (xy 106.721972 95.165365)
+					(xy 106.735136 95.178358) (xy 106.76732 95.21901) (xy 106.790926 95.2622) (xy 106.798395 95.280207)
+					(xy 106.812944 95.329282) (xy 106.820075 95.380857) (xy 106.820865 95.405503) (xy 106.81746 95.456191)
+					(xy 106.805976 95.507602) (xy 106.792045 95.543501) (xy 106.767441 95.587258) (xy 106.736861 95.626207)
+					(xy 106.713154 95.649502) (xy 106.673175 95.679842) (xy 106.627974 95.704548) (xy 106.594941 95.71789)
+					(xy 106.547024 95.731657) (xy 106.496971 95.739709) (xy 106.449616 95.74207) (xy 106.396706 95.739155)
+					(xy 106.346452 95.73041) (xy 106.30307 95.717402) (xy 106.254951 95.696015) (xy 106.211708 95.668858)
+					(xy 106.18559 95.647548) (xy 106.151174 95.611186) (xy 106.122666 95.569879) (xy 106.106943 95.539593)
+					(xy 106.089381 95.49042) (xy 106.080402 95.441664) (xy 106.078123 95.399153) (xy 106.078169 95.398176)
+					(xy 106.289149 95.398176) (xy 106.296445 95.449317) (xy 106.320621 95.495826) (xy 106.333356 95.510284)
+					(xy 106.373989 95.538907) (xy 106.42365 95.552937) (xy 106.449616 95.554492) (xy 106.499442 95.548275)
+					(xy 106.544737 95.527509) (xy 106.565387 95.510284) (xy 106.594168 95.470337) (xy 106.608277 95.422731)
+					(xy 106.609839 95.398176) (xy 106.602503 95.347076) (xy 106.578193 95.3007) (xy 106.565387 95.286313)
+					(xy 106.524954 95.257532) (xy 106.475491 95.243423) (xy 106.449616 95.241861) (xy 106.399607 95.248112)
+					(xy 106.354113 95.268992) (xy 106.333356 95.286313) (xy 106.304734 95.326102) (xy 106.290703 95.37363)
+					(xy 106.289149 95.398176) (xy 106.078169 95.398176) (xy 106.080565 95.34774) (xy 106.087892 95.300967)
+					(xy 106.10109 95.252582) (xy 106.114026 95.217192) (xy 106.135149 95.171498) (xy 106.151884 95.141721)
+					(xy 106.178676 95.098107) (xy 106.197802 95.067471) (xy 106.415666 94.72602) (xy 106.673098 94.72602)
 				)
 			)
@@
 		(net 30)
 	)
+	(zone
+		(net 0)
+		(net_name "")
+		(layers "F&B.Cu")
+		(hatch edge 0.5)
+		(connect_pads
+			(clearance 0.5)
+		)
+		(min_thickness 0.25)
+		(filled_areas_thickness no)
+		(fill yes
+			(thermal_gap 0.5)
+			(thermal_bridge_width 0.5)
+			(island_removal_mode 1)
+			(island_area_min 10)
+		)
+		(polygon
+			(pts
+				(xy 24.373343 137.896439) (xy 23.773343 21.096439) (xy 163.073343 20.296439) (xy 163.573343 135.496439)
+			)
+		)
+	)
 	(group ""
