File: pcb/pcb.kicad_pcb (KiCad board)
At the start: 2 copper layers, 118.8 x 99.7 mm, 43 parts, among them J1 BAT, U1 xiao-ble

Commit message: rename to Charma
Parts:
- DL1, DL10, DL11, DL12, DL13, DL14, DL15, DL16, DL17, DL18, DL2, DL3, DL4, DL5, DL6, DL7, DL8, DL9: footprint karmalib:Diode_SOD123 -> charmalib:Diode_SOD123
- RSW1: footprint karmalib:SKHLLCA010 -> charmalib:SKHLLCA010
- SWL1, SWL10, SWL11, SWL12, SWL13, SWL14, SWL15, SWL16, SWL17, SWL18, SWL2, SWL3, SWL4, SWL5, SWL6, SWL7, SWL8, SWL9: footprint karmalib:Kailh_Socket_PG1350_Optional -> charmalib:Kailh_Socket_PG1350_Optional
- U1: footprint karmalib:XIAO_nRF52840_SMD_Cutout -> charmalib:XIAO_nRF52840_SMD_Cutout

Commit message: Parameterise
Parts:
- added DR1: D_Small, charmalib:Diode_SOD123, F.Cu at (226.0, 41.8)
- added DR10: D_Small, charmalib:Diode_SOD123, F.Cu at (253.5, 96.5)
- added DR11: D_Small, charmalib:Diode_SOD123, F.Cu at (253.5, 99.0)
- added DR12: D_Small, charmalib:Diode_SOD123, F.Cu at (253.5, 101.6)
- added DR13: D_Small, charmalib:Diode_SOD123, F.Cu at (259.7, 88.8)
- added DR14: D_Small, charmalib:Diode_SOD123, F.Cu at (259.7, 91.4)
- added DR15: D_Small, charmalib:Diode_SOD123, F.Cu at (259.7, 93.9)
- added DR16: D_Small, charmalib:Diode_SOD123, F.Cu at (259.7, 96.5)
- added DR17: D_Small, charmalib:Diode_SOD123, F.Cu at (259.7, 99.0)
- added DR18: D_Small, charmalib:Diode_SOD123, F.Cu at (259.7, 101.6)
- added DR2: D_Small, charmalib:Diode_SOD123, F.Cu at (247.3, 91.4)
- added DR3: D_Small, charmalib:Diode_SOD123, F.Cu at (247.3, 93.9)
- added DR4: D_Small, charmalib:Diode_SOD123, F.Cu at (247.3, 96.5)
- added DR5: D_Small, charmalib:Diode_SOD123, F.Cu at (247.3, 99.0)
- added DR6: D_Small, charmalib:Diode_SOD123, F.Cu at (247.3, 101.6)
- added DR7: D_Small, charmalib:Diode_SOD123, F.Cu at (253.5, 88.8)
- added DR8: D_Small, charmalib:Diode_SOD123, F.Cu at (253.5, 91.4)
- added DR9: D_Small, charmalib:Diode_SOD123, F.Cu at (253.5, 93.9)
- added JR1: BAT, Connector_PinHeader_2.54mm:PinHeader_1x02_P2.54mm_Vertical, F.Cu at (265.1, 89.9)
- added MCUR1: xiao-ble, charmalib:XIAO_nRF52840_SMD_Cutout, F.Cu at (196.5, 63.8)
- added RSWR1: SW_Push, Button_Switch_SMD:SW_Push_1P1T-MP_NO_Horizontal_Alps_SKRTLAE010, F.Cu at (270.7, 90.1)
- added SWR1: SW_Push_45deg, charmalib:Kailh_Socket_PG1350_Optional, F.Cu at (225.3, 34.2)
- added SWR10: SW_Push_45deg, charmalib:Kailh_Socket_PG1350_Optional, F.Cu at (278.2, 52.3)
- added SWR11: SW_Push_45deg, charmalib:Kailh_Socket_PG1350_Optional, F.Cu at (295.9, 52.3)
- added SWR12: SW_Push_45deg, charmalib:Kailh_Socket_PG1350_Optional, F.Cu at (313.6, 52.3)
- added SWR13: SW_Push_45deg, charmalib:Kailh_Socket_PG1350_Optional, F.Cu at (225.3, 70.3)
- added SWR14: SW_Push_45deg, charmalib:Kailh_Socket_PG1350_Optional, F.Cu at (242.9, 70.3)
- added SWR15: SW_Push_45deg, charmalib:Kailh_Socket_PG1350_Optional, F.Cu at (260.6, 70.3)
- added SWR16: SW_Push_45deg, charmalib:Kailh_Socket_PG1350_Optional, F.Cu at (278.2, 70.3)
- added SWR17: SW_Push_45deg, charmalib:Kailh_Socket_PG1350_Optional, F.Cu at (295.9, 70.3)
- added SWR18: SW_Push_45deg, charmalib:Kailh_Socket_PG1350_Optional, F.Cu at (313.6, 70.3)
- added SWR2: SW_Push_45deg, charmalib:Kailh_Socket_PG1350_Optional, F.Cu at (242.9, 34.2)
- added SWR3: SW_Push_45deg, charmalib:Kailh_Socket_PG1350_Optional, F.Cu at (260.6, 34.2)
- added SWR4: SW_Push_45deg, charmalib:Kailh_Socket_PG1350_Optional, F.Cu at (278.2, 34.2)
- added SWR5: SW_Push_45deg, charmalib:Kailh_Socket_PG1350_Optional, F.Cu at (295.9, 34.2)
- added SWR6: SW_Push_45deg, charmalib:Kailh_Socket_PG1350_Optional, F.Cu at (313.6, 34.2)
- added SWR7: SW_Push_45deg, charmalib:Kailh_Socket_PG1350_Optional, F.Cu at (225.3, 52.3)
- added SWR8: SW_Push_45deg, charmalib:Kailh_Socket_PG1350_Optional, F.Cu at (242.9, 52.3)
- added SWR9: SW_Push_45deg, charmalib:Kailh_Socket_PG1350_Optional, F.Cu at (260.6, 52.3)
- RSWL1: renamed from RSW1; footprint charmalib:SKHLLCA010 -> Button_Switch_SMD:SW_Push_1P1T-MP_NO_Horizontal_Alps_SKRTLAE010
- moved RSWL1 52.0 mm to (63.5, 31.9), turned to 180 degrees
- renumbered J1 to JL1, U1 to MCUL1
Routing:
- net GND_L: track 195.3 -> 47.9 mm
- net RESET_L: track 88.0 -> 34.3 mm
Other:
- board text added: "BAT"

Commit message: Update refs
Parts:
- added HOLER1: MountingHole_2.2mm_M2_DIN965_Pad, MountingHole:MountingHole_2.2mm_M2_DIN965_Pad, F.Cu at (351.5, 38.4)
- added HOLER2: MountingHole_2.2mm_M2_DIN965_Pad, MountingHole:MountingHole_2.2mm_M2_DIN965_Pad, F.Cu at (422.8, 38.4)
- added HOLER3: MountingHole_2.2mm_M2_DIN965_Pad, MountingHole:MountingHole_2.2mm_M2_DIN965_Pad, F.Cu at (327.8, 112.6)
- added HOLER4: MountingHole_2.2mm_M2_DIN965_Pad, MountingHole:MountingHole_2.2mm_M2_DIN965_Pad, F.Cu at (422.8, 96.9)
- renumbered topleft to HOLEL1, topright to HOLEL2, bottomleft to HOLEL3, bottomright to HOLEL4

Commit message: Diode orientation
Parts:
- moved HOLER4 253.8 mm to (171.5, 61.0)
- moved HOLER1 183.6 mm to (171.5, 2.50)
- moved HOLER2 183.6 mm to (242.8, 2.50)
- moved SWR18 151.1 mm to (163.3, 86.9), turned to -42 degrees
- moved SWR6 130.3 mm to (183.2, 33.8)
- moved SWR17 115.1 mm to (180.9, 76.1), turned to -21 degrees
- moved SWR11 112.7 mm to (183.2, 50.8)
- moved SWR12 112.4 mm to (201.2, 48.2)
- moved HOLEL2 105.6 mm to (26.2, 2.50)
- moved DR18 105.6 mm to (155.0, 87.3), turned to -42 degrees
- moved DR6 101.5 mm to (176.8, 28.6)
- moved DR2 97.7 mm to (194.8, 9.05)
- moved DR3 95.6 mm to (212.8, 4.80)
- moved RSWR1 95.0 mm to (235.5, 1.95)
- moved DR11 93.5 mm to (176.8, 45.6)
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- renumbered JL1 to BATL1, JR1 to BATR1, MCUR1 to MCUR2
Routing:
- net Net-(DL9-A): track 7.65 -> 318.2 mm, vias 0 -> 2
- net COL4_L: track 167.1 -> 0.00 mm
- net Net-(DL18-A): track 7.82 -> 171.4 mm, vias 0 -> 3
- net COL3_L: track 143.5 -> 15.8 mm, vias 2 -> 0
- net ROW2_L: track 119.4 -> 0.00 mm, vias 5 -> 0
- net ROW0_L: track 82.3 -> 0.00 mm
- net Net-(DL13-A): track 8.04 -> 82.3 mm
- net Net-(DL14-A): track 7.65 -> 63.8 mm
- net GND_L: track 47.9 -> 0.00 mm, vias 1 -> 0
- net ROW3_L: track 163.6 -> 119.4 mm, vias 3 -> 5
- net ROW1_L: track 108.1 -> 82.0 mm
- net COL1_L: track 56.1 -> 74.1 mm, vias 0 -> 1
- net COL2_L: track 121.7 -> 129.8 mm
- net Net-(DL3-A): track 8.04 -> 0.00 mm
- net Net-(DL8-A): track 7.72 -> 0.00 mm

Commit message: Add origin offset to place inside edge cuts
Parts:
- turned BATL1 to 90 degrees
- turned BATR1 to -90 degrees
- turned DL1 to -90 degrees
- turned DL10 to -90 degrees
- turned DL11 to -90 degrees
- turned DL12 to -90 degrees
- turned DL13 to -90 degrees
- turned DL14 to -90 degrees
- turned DL15 to -90 degrees
- turned DL16 to -90 degrees
- turned DL17 to -111 degrees
- turned DL18 to -132 degrees
- turned DL2 to -90 degrees
- turned DL3 to -90 degrees
- turned DL4 to -90 degrees
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- renumbered MCUR2 to MCUR1
Routing:
- net ROW3_L: track 119.4 -> 0.00 mm, vias 5 -> 0
- net Net-(DL17-A): track 9.10 -> 128.5 mm, vias 0 -> 5
- net GND_L: track 0.00 -> 52.5 mm
- net COL0_L: track 52.5 -> 0.00 mm
- net RESET_L: track 34.3 -> 0.00 mm
- net Net-(DL13-A): track 82.3 -> 116.6 mm
- net Net-(DL14-A): track 63.8 -> 56.1 mm
- net COL3_L: track 15.8 -> 23.4 mm
