File: pcb/pcb.kicad_pcb (KiCad board)
At the start: 2 copper layers, 118.8 x 99.7 mm, 86 parts

Commit message: Use SKQB for reset
Parts:
- RSWL1, RSWR1: footprint Button_Switch_SMD:SW_Push_1P1T-MP_NO_Horizontal_Alps_SKRTLAE010 -> Button_Switch_SMD:SW_SPST_SKQG_WithStem
- moved DL15 42.4 mm to (109.2, 75.6)
- moved DR11 42.4 mm to (206.8, 75.6)
- moved DL1 42.4 mm to (37.2, 53.5)
- moved DL10 42.4 mm to (109.2, 58.6)
- moved DL11 42.4 mm to (37.2, 87.5)
- moved DL12 42.4 mm to (55.2, 73.0)
- moved DL13 42.4 mm to (73.2, 68.8)
- moved DL14 42.4 mm to (91.2, 73.0)
- moved DL16 42.4 mm to (91.2, 97.1)
- moved DL17 42.4 mm to (113.8, 98.9)
- moved DL18 42.4 mm to (134.3, 108.6)
- moved DL5 42.4 mm to (109.2, 41.6)
- moved DL6 42.4 mm to (37.2, 70.5)
- moved DR1 42.4 mm to (206.8, 41.6)
- moved DR10 42.4 mm to (278.8, 70.5)
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- renumbered MCUR1 to MCUR2
Routing:
- net Net-(DL9-A): track 318.2 -> 151.1 mm
- net COL4_L: track 0.00 -> 167.1 mm
- net ROW3_L: track 0.00 -> 163.6 mm, vias 0 -> 3
- net Net-(DL18-A): track 171.4 -> 7.82 mm, vias 3 -> 0
- net COL0_L: track 0.00 -> 52.5 mm
- net Net-(DL14-A): track 56.1 -> 7.65 mm
- net RESET_L: track 0.00 -> 28.8 mm
- net Net-(DL13-A): track 116.6 -> 90.4 mm
- net ROW1_L: track 82.0 -> 108.1 mm
- net COL3_L: track 23.4 -> 0.00 mm
- net COL1_L: track 74.1 -> 56.1 mm, vias 1 -> 0
- net GND_L: track 52.5 -> 42.0 mm, vias 0 -> 1
- net COL2_L: track 129.8 -> 121.7 mm
- net Net-(DL3-A): track 0.00 -> 8.04 mm
- net Net-(DL8-A): track 0.00 -> 7.72 mm

Commit message: Postion tweaks to match edge cuts
Parts:
- moved RSWL1 1.25 mm to (64.0, 33.1)
- moved RSWR1 1.25 mm to (265.0, 33.1)
- moved DL1 0.35 mm to (37.5, 53.8)
- moved DL10 0.35 mm to (109.5, 58.9)
- moved DL11 0.35 mm to (37.5, 87.8)
- moved DL12 0.35 mm to (55.5, 73.3)
- moved DL13 0.35 mm to (73.5, 69.0)
- moved DL14 0.35 mm to (91.5, 73.3)
- moved DL15 0.35 mm to (109.5, 75.8)
- moved DL2 0.35 mm to (55.5, 39.3)
- moved DL3 0.35 mm to (73.5, 35.0)
- moved DL4 0.35 mm to (91.5, 39.3)
- moved DL5 0.35 mm to (109.5, 41.9)
- moved DL6 0.35 mm to (37.5, 70.8)
- moved DL7 0.35 mm to (55.5, 56.3)
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
Commit message: Move MCU closer to edge
Parts:
- moved HOLER4 25.3 mm to (176.2, 91.3)
- moved BATR1 25.0 mm to (227.3, 86.3)
- moved DR1 25.0 mm to (181.5, 41.9)
- moved DR10 25.0 mm to (253.5, 70.8)
- moved DR11 25.0 mm to (181.5, 75.8)
- moved DR12 25.0 mm to (199.5, 73.3)
- moved DR13 25.0 mm to (217.5, 69.0)
- moved DR14 25.0 mm to (235.5, 73.3)
- moved DR15 25.0 mm to (253.5, 87.8)
- moved DR16 25.0 mm to (199.5, 97.1)
- moved DR17 25.0 mm to (177.8, 103.5)
- moved DR18 25.0 mm to (159.8, 117.3)
- moved DR2 25.0 mm to (199.5, 39.3)
- moved DR3 25.0 mm to (217.5, 35.0)
- moved DR4 25.0 mm to (235.5, 39.3)
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- renumbered MCUR2 to MCUR1

Commit message: Update placement
Parts:
- moved MCUR1 25.0 mm to (263.5, 39.7)
Changed lines of the file:
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@@
 		(legacy_teardrops no)
 	)
-	(paper "User" 500 200)
+	(paper "User" 300 200)
 	(title_block
 		(title "Charma Wireless Split Keyboard")
@@
 	(footprint "charmalib:XIAO_nRF52840_SMD_Cutout"
 		(layer "F.Cu")
-		(at 288.5 40.39 -90)
+		(at 263.5 39.7 -90)
 		(property "Reference" "MCUR1"
 			(at -19.3989 -11.28268 90)

Commit message: tweaks
Parts:
- moved DL4 70.3 mm to (159.5, 21.7)
- moved SWL4 29.1 mm to (114.7, 20.7)
Routing:
- net COL4_L: track 167.1 -> 0.00 mm
- net ROW3_L: track 163.6 -> 0.00 mm, vias 3 -> 0
- net Net-(DL9-A): track 151.1 -> 0.00 mm, vias 2 -> 0
- net Net-(DL17-A): track 128.5 -> 0.00 mm, vias 5 -> 0
- net COL2_L: track 121.7 -> 0.00 mm, vias 1 -> 0
- net ROW1_L: track 108.1 -> 0.00 mm, vias 4 -> 0
- net Net-(DL13-A): track 90.4 -> 0.00 mm
- net VBAT_L: track 88.5 -> 0.00 mm
- net COL1_L: track 56.1 -> 0.00 mm
- net COL0_L: track 52.5 -> 0.00 mm
- net GND_L: track 42.0 -> 0.00 mm, vias 1 -> 0
- net RESET_L: track 28.8 -> 0.00 mm
- net Net-(DL10-A): track 8.11 -> 0.00 mm
- net Net-(DL5-A): track 8.09 -> 0.00 mm
- net Net-(DL4-A): track 8.04 -> 0.00 mm
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
Commit message: hairline
Parts:
- moved DL4 70.3 mm to (91.5, 39.3)
- moved SWL4 29.1 mm to (98.0, 44.5)
- moved BATR1 3.00 mm to (230.3, 86.3)
- moved DR1 3.00 mm to (184.5, 41.9)
- moved DR10 3.00 mm to (256.5, 70.8)
- moved DR11 3.00 mm to (184.5, 75.8)
- moved DR12 3.00 mm to (202.5, 73.3)
- moved DR13 3.00 mm to (220.5, 69.0)
- moved DR14 3.00 mm to (238.5, 73.3)
- moved DR15 3.00 mm to (256.5, 87.8)
- moved DR16 3.00 mm to (202.5, 97.1)
- moved DR17 3.00 mm to (180.8, 103.5)
- moved DR18 3.00 mm to (162.8, 117.3)
- moved DR2 3.00 mm to (202.5, 39.3)
- moved DR3 3.00 mm to (220.5, 35.0)
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
Commit message: Use socketed Xiao
Parts:
- added MCUL1: SeeeduinoXIAO nRF52840, charmalib:XIAO nRF52840 Socketed w pogo, F.Cu at (40.5, 39.7)
- added MCUR1: SeeeduinoXIAO nRF52840, charmalib:XIAO nRF52840 Socketed w pogo, F.Cu at (266.5, 39.7)

Commit message: Fix diodes
Parts:
- removed the MCUL1 at (40.5, 39.7)
- removed the MCUR1 at (266.5, 39.7)
- DR1, DR10, DR11, DR12, DR13, DR14, DR15, DR16, DR17, DR18, DR2, DR3, DR4, DR5, DR6, DR7, DR8, DR9, RSWL1, RSWR1: moved to B.Cu
- turned RSWL1 to 0 degrees
- turned RSWR1 to 0 degrees
Other:
- board size 118.8 x 99.7 mm -> 247.1 x 99.7 mm
