File: pcb/pcb.kicad_pcb (KiCad board)
At the start: 2 copper layers, 248 x 100.9 mm, 92 parts

Commit message: Position power switches
Parts:
- moved RSWL1 63.9 mm to (64.0, 33.1)
- moved PSWL1 39.2 mm to (33.5, 54.8), turned to -90 degrees
- moved MCUL1 4.79 mm to (40.0, 39.0)
- moved PSWR1 2.95 mm to (274.4, 54.8)
Routing:
- net VBAT_R: track 83.3 -> 79.2 mm
- net MCU_BAT+_R: track 23.0 -> 26.1 mm
- net GND_R: track 140.5 -> 139.9 mm

Commit message: Position power switches
Parts:
- moved PSWL1 1.51 mm to (33.8, 56.2)
- moved PSWR1 1.51 mm to (274.2, 56.2)
Changed lines of the file:
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@@
 	(footprint "Button_Switch_SMD:SW_SPDT_PCM12"
 		(layer "F.Cu")
-		(at 33.549999 54.75 -90)
+		(at 33.75 56.25 -90)
 		(descr "Ultraminiature Surface Mount Slide Switch, right-angle, https://www.ckswitches.com/media/1424/pcm.pdf")
 		(property "Reference" "PSWL1"
@@
 	(footprint "Button_Switch_SMD:SW_SPDT_PCM12"
 		(layer "F.Cu")
-		(at 274.45 54.75 90)
+		(at 274.25 56.25 90)
 		(descr "Ultraminiature Surface Mount Slide Switch, right-angle, https://www.ckswitches.com/media/1424/pcm.pdf")
 		(property "Reference" "PSWR1"

Commit message: Route and silkscreen
Parts:
- REF** (x4): footprint kbd:Breakaway_Tabs -> charmalib:Breakaway_Tabs
Connections:
- MCUR1 pad 1: ROW3_R -> unconnected-(MCUR1-PA02_A0_D0-Pad1)
- MCUR1 pad 10: COL3_R -> ROW2_R
- MCUR1 pad 11: COL2_R -> ROW3_R
- MCUR1 pad 2: ROW2_R -> unconnected-(MCUR1-PA4_A1_D1-Pad2)
- MCUR1 pad 3: ROW1_R -> COL4_R
- MCUR1 pad 4: ROW0_R -> COL3_R
- MCUR1 pad 5: COL0_R -> COL2_R
- MCUR1 pad 7: unconnected-(MCUR1-PB08_A6_D6_TX-Pad7) -> COL0_R
- MCUR1 pad 8: unconnected-(MCUR1-PB09_A7_D7_RX-Pad8) -> ROW0_R
- MCUR1 pad 9: COL4_R -> ROW1_R
- RSWL1 pad 1: RESET_L -> GND_L
- RSWL1 pad 2: GND_L -> RESET_L
Routing:
- net COL4_L: track 0.00 -> 166.5 mm, vias 0 -> 1
- net ROW3_L: track 0.00 -> 164.1 mm, vias 0 -> 3
- net COL3_L: track 0.00 -> 141.9 mm, vias 0 -> 1
- net ROW2_R: track 0.00 -> 122.7 mm, vias 0 -> 5
- net COL2_L: track 0.00 -> 122.3 mm, vias 0 -> 1
- net ROW2_L: track 0.00 -> 117.8 mm, vias 0 -> 5
- net COL0_R: track 34.0 -> 150.1 mm
- net ROW1_L: track 0.00 -> 99.7 mm, vias 0 -> 5
- net GND_L: track 0.00 -> 97.7 mm
- net ROW3_R: track 49.4 -> 143.3 mm, vias 0 -> 3
- net COL1_R: track 34.0 -> 127.8 mm
- net ROW0_L: track 0.00 -> 85.0 mm, vias 0 -> 4
- net COL2_R: track 34.0 -> 117.3 mm
- net VBAT_L: track 0.00 -> 76.8 mm
- net COL1_L: track 0.00 -> 58.2 mm
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Other:
- board text removed: "RST"
